File: hardware/cm5.kicad_sch (KiCad schematic)
At the start: 1 part

Commit message: Fix schematic connectivity and add flashing access
The camera and Ethernet buses now connect across sheets: they use
unnamed bus groups so the member nets keep their names. Ethernet pair 2
negative is no longer tied to GND.

The RP2354A core supply reaches the regulator output, and a 12 MHz
crystal drives XIN/XOUT, which USB and the USB bootloader need. The
CM5 gets GPIO_VREF on 3.3 V, the IO Board's boot and EEPROM jumper
header, and a data-only USB-C port with 5.1 kOhm CC resistors for
flashing the eMMC.

Co-Authored-By: Claude Opus 5.5 <noreply@anthropic.com>
Parts:
- added C22, C23: 100n, Capacitor_SMD:C_0402_1005Metric, symbol Device:C
- added J7: Conn_02x07_Odd_Even, Connector_PinHeader_2.54mm:PinHeader_2x07_P2.54mm_Vertical, symbol Connector_Generic:Conn_02x07_Odd_Even
Connections:
- net +3.3V: now also Module1.78 (GPIO_VREF(1.8v/3.3v_Input))
- net +5V: now also C22.1, C23.1
- net GND: now also C22.2, C23.2, J7.1 (Pin_1), J7.11 (Pin_11), J7.13 (Pin_13), J7.3 (Pin_3), J7.5 (Pin_5), J7.7 (Pin_7), J7.9 (Pin_9); no longer Module1.9 (Ethernet_Pair2_N)
- net USBOTG: now reaches Module1.101 (USB_OTG_ID)
- net USBOTG: now also J7.10 (Pin_10)
- net USB2_N: now reaches Module1.103 (USB2_N)
- net USB2_P: now reaches Module1.105 (USB2_P)
- net SYNC_OUT: now reaches Module1.18 (Ethernet_SYNC_OUT(3.3v))
- net SYNC_OUT: now also J7.6 (Pin_6)
- net EEPROM_nWP: now reaches Module1.20 (EEPROM_nWP)
- net EEPROM_nWP: now also J7.4 (Pin_4)
- net PWR_BUT: now reaches Module1.92 (PWR_BUT)
- net PWR_BUT: now also J7.14 (Pin_14)
- net nRPIBOOT: now reaches Module1.93 (nRPIBOOT)
- net nRPIBOOT: now also J7.2 (Pin_2)
- net CC1: now reaches Module1.94 (CC1)
- net CC2: now reaches Module1.96 (CC2)
- net PMIC_ENABLE: now reaches Module1.99 (PMIC_ENABLE)
- net PMIC_ENABLE: now also J7.12 (Pin_12)
- new net TRD2_N: Module1.9 (Ethernet_Pair2_N)
- no-connect marks 45 -> 64
Other:
- note added: "Configuration Jumper"
- note added: "Decoupling"
- moved on the sheet: Module1A
