File: hardware/cm5.kicad_sch (KiCad schematic)
At the start: 8 parts, among them J7 Conn_02x07_Odd_Even, J9 Conn_02x08_Odd_Even

Commit message: Add LCSC part numbers and links, fix J7 part number
- Every part found on LCSC gets an "LCSC PN" (C-number) and an "LCSC" product
  link field, in the schematic and on the PCB footprints. Exact matches where
  LCSC lists the part; equivalents with the same specs where it does not or
  has no stock (C46, C26/C28/C30/C33/C34/C40, C29, C31, R6/R7, R21, R24,
  J3/J4, J7/J9/J13). Left empty: IC3, IC5 (not on LCSC), IC10, IC12
  (JLCPCB-only listings).
- J7: the MPN 61301421121 is a 2.54 mm header, but the footprint is 1.27 mm.
  Now Wurth 62201421121 (WR-PHD 1.27 mm 2x7) with matching description,
  datasheet and Mouser fields.
- Interactive HTML BOM in hardware/bom; KiCad project file re-saved.

Co-Authored-By: Claude Opus 5.5 <noreply@anthropic.com>
Claude-Session: https://claude.ai/code/session_01AhLYztcZikG9g81njGtEr1
Parts:
- C22, C23, C43: LCSC (none) -> https://www.lcsc.com/product-detail/C71629.html; LCSC PN (none) -> C71629
- C41: LCSC (none) -> https://www.lcsc.com/product-detail/C84494.html; LCSC PN (none) -> C84494
- C42: LCSC (none) -> https://www.lcsc.com/product-detail/C19702.html; LCSC PN (none) -> C19702
- J7: LCSC (none) -> https://www.lcsc.com/product-detail/C22438122.html; LCSC PN (none) -> C22438122; MPN 61301421121 -> 62201421121; Mouser https://www.mouser.com/ProductDetail/710-61301421121 -> https://www.mouser.com/ProductDetail/710-62201421121; Mouser PN 710-61301421121 -> 710-62201421121
- J9: LCSC (none) -> https://www.lcsc.com/product-detail/C22438123.html; LCSC PN (none) -> C22438123
- Module1: LCSC (none) -> https://www.lcsc.com/product-detail/C6782225.html; LCSC PN (none) -> C6782225
Changed lines of the file:
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@@
+			)
+		)
+		(property "LCSC PN" "C19702"
+			(at 19.05 57.15 0)
+			(hide yes)
+			(show_name no)
+			(do_not_autoplace no)
+			(effects
+				(font
+					(size 1.27 1.27)
+				)
+			)
+		)
+		(property "LCSC" "https://www.lcsc.com/product-detail/C19702.html"
+			(at 19.05 57.15 0)
+			(hide yes)
+			(show_name no)
+			(do_not_autoplace no)
+			(effects
+				(font
+					(size 1.27 1.27)
+				)
 			)
 		)
@@
 			)
 		)
+		(property "LCSC PN" "C6782225"
+			(at 81.28 88.9 0)
+			(hide yes)
+			(show_name no)
+			(do_not_autoplace no)
+			(effects
+				(font
+					(size 1.27 1.27)
+				)
+			)
+		)
+		(property "LCSC" "https://www.lcsc.com/product-detail/C6782225.html"
+			(at 81.28 88.9 0)
+			(hide yes)
+			(show_name no)
+			(do_not_autoplace no)
+			(effects
+				(font
+					(size 1.27 1.27)
+				)
+			)
+		)
 		(property "Note" "2 pcs per board (both CM5 connectors). CM5 module (eMMC variant) ordered separately."
 			(at 81.28 88.9 0)
@@
 			)
 		)
+		(property "LCSC PN" "C71629"
+			(at 29.21 57.15 0)
+			(hide yes)
+			(show_name no)
+			(do_not_autoplace no)
+			(effects
+				(font
+					(size 1.27 1.27)
+				)
+			)
+		)
+		(property "LCSC" "https://www.lcsc.com/product-detail/C71629.html"
+			(at 29.21 57.15 0)
+			(hide yes)
+			(show_name no)
+			(do_not_autoplace no)
+			(effects
+				(font
+					(size 1.27 1.27)
+				)
+			)
+		)
 		(pin "1"
 		)
@@
 		)
 		(property "Mouser" "https://www.mouser.com/ProductDetail/81-GRM155R71C104KA88"
+			(at 31.75 31.75 0)
+			(hide yes)
+			(show_name no)
+			(do_not_autoplace no)
+			(effects
+				(font
+					(size 1.27 1.27)
+				)
+			)
+		)
+		(property "LCSC PN" "C71629"
+			(at 31.75 31.75 0)
+			(hide yes)
+			(show_name no)
+			(do_not_autoplace no)
+			(effects
+				(font
+					(size 1.27 1.27)
+				)
+			)
+		)
+		(property "LCSC" "https://www.lcsc.com/product-detail/C71629.html"
 			(at 31.75 31.75 0)
 			(hide yes)
@@
 			)
 		)
+		(property "LCSC PN" "C22438123"
+			(at 34.29 132.08 0)
+			(hide yes)
+			(show_name no)
+			(do_not_autoplace no)
+			(effects
+				(font
+					(size 1.27 1.27)
+				)
+			)
+		)
+		(property "LCSC" "https://www.lcsc.com/product-detail/C22438123.html"
+			(at 34.29 132.08 0)
+			(hide yes)
+			(show_name no)
+			(do_not_autoplace no)
+			(effects
+				(font
+					(size 1.27 1.27)
+				)
+			)
+		)
 		(property "Description" "Generic connector, double row, 02x08, odd/even pin numbering scheme (row 1 odd numbers, row 2 even numbers), script generated (kicad-library-utils/schlib/autogen/connector/)"
 			(at 34.29 132.08 0)
@@
 			)
 		)
-		(property "Datasheet" "https://www.we-online.com/components/products/datasheet/61301421121.pdf"
+		(property "Datasheet" "https://www.we-online.com/components/products/datasheet/62201421121.pdf"
 			(at 30.48 91.44 0)
 			(hide yes)
@@
 			)
 		)
-		(property "Description" "CONN HDR 2x7 2.54mm vertical THT"
+		(property "Description" "CONN HDR 2x7 1.27mm vertical THT"
 			(at 30.48 91.44 0)
 			(hide yes)
@@
 			)
 		)
-		(property "MPN" "61301421121"
+		(property "MPN" "62201421121"
 			(at 30.48 91.44 0)
 			(hide yes)
@@
 			)
 		)
-		(property "Mouser PN" "710-61301421121"
+		(property "Mouser PN" "710-62201421121"
 			(at 30.48 91.44 0)
 			(hide yes)
@@
 			)
 		)
-		(property "Mouser" "https://www.mouser.com/ProductDetail/710-61301421121"
+		(property "Mouser" "https://www.mouser.com/ProductDetail/710-62201421121"
+			(at 30.48 91.44 0)
+			(hide yes)
+			(show_name no)
+			(do_not_autoplace no)
+			(effects
+				(font
+					(size 1.27 1.27)
+				)
+			)
+		)
+		(property "LCSC PN" "C22438122"
+			(at 30.48 91.44 0)
+			(hide yes)
+			(show_name no)
+			(do_not_autoplace no)
+			(effects
+				(font
+					(size 1.27 1.27)
+				)
+			)
+		)
+		(property "LCSC" "https://www.lcsc.com/product-detail/C22438122.html"
 			(at 30.48 91.44 0)
 			(hide yes)
@@
 			)
 		)
+		(property "LCSC PN" "C6782225"
+			(at 116.84 83.82 0)
+			(hide yes)
+			(show_name no)
+			(do_not_autoplace no)
+			(effects
+				(font
+					(size 1.27 1.27)
+				)
+			)
+		)
+		(property "LCSC" "https://www.lcsc.com/product-detail/C6782225.html"
+			(at 116.84 83.82 0)
+			(hide yes)
+			(show_name no)
+			(do_not_autoplace no)
+			(effects
+				(font
+					(size 1.27 1.27)
+				)
+			)
+		)
 		(property "Note" "2 pcs per board (both CM5 connectors). CM5 module (eMMC variant) ordered separately."
 			(at 116.84 83.82 0)
@@
 			)
 		)
+		(property "LCSC PN" "C71629"
+			(at 19.05 31.75 0)
+			(hide yes)
+			(show_name no)
+			(do_not_autoplace no)
+			(effects
+				(font
+					(size 1.27 1.27)
+				)
+			)
+		)
+		(property "LCSC" "https://www.lcsc.com/product-detail/C71629.html"
+			(at 19.05 31.75 0)
+			(hide yes)
+			(show_name no)
+			(do_not_autoplace no)
+			(effects
+				(font
+					(size 1.27 1.27)
+				)
+			)
+		)
 		(pin "1"
 		)
@@
 			(at 43.18 31.75 0)
 			(hide yes)
+			(show_name no)
+			(do_not_autoplace no)
+			(effects
+				(font
+					(size 1.27 1.27)
+				)
+			)
+		)
+		(property "LCSC PN" "C84494"
+			(at 43.18 31.75 0)
+			(hide yes)
+			(show_name no)
+			(do_not_autoplace no)
+			(effects
+				(font
+					(size 1.27 1.27)
+				)
+			)
+		)
+		(property "LCSC" "https://www.lcsc.com/product-detail/C84494.html"
+			(at 43.18 31.75 0)
+			(hide yes)
