File: hardware/ethernet.kicad_sch (KiCad schematic)
At the start: 7 parts, among them J9 THD-02-R, U1 TPD4EUSB30, U2 TPD4EUSB30, U3 MagJack-A70-112-331N126

Commit message: Fix schematic connectivity and add flashing access
The camera and Ethernet buses now connect across sheets: they use
unnamed bus groups so the member nets keep their names. Ethernet pair 2
negative is no longer tied to GND.

The RP2354A core supply reaches the regulator output, and a 12 MHz
crystal drives XIN/XOUT, which USB and the USB bootloader need. The
CM5 gets GPIO_VREF on 3.3 V, the IO Board's boot and EEPROM jumper
header, and a data-only USB-C port with 5.1 kOhm CC resistors for
flashing the eMMC.

Co-Authored-By: Claude Opus 5.5 <noreply@anthropic.com>
Connections:
- net ETH0.TRD0_N is gone; now on net TRD0_N: U2.4 (D2+), U2.7
- net ETH0.TRD0_P is gone; now on net TRD0_P: U2.5 (D2-), U2.6
- net ETH0.TRD1_N is gone; now on net TRD1_N: U2.2 (D1-), U2.9
- net ETH0.TRD1_P is gone; now on net TRD1_P: U2.1 (D1+), U2.10
- net ETH0.TRD2_N is gone; now on net TRD2_N: U1.4 (D2+), U1.7
- net ETH0.TRD2_P is gone; now on net TRD2_P: U1.5 (D2-), U1.6
- net ETH0.TRD3_N is gone; now on net TRD3_N: U1.2 (D1-), U1.9
- net ETH0.TRD3_P is gone; now on net TRD3_P: U1.1 (D1+), U1.10
Changed lines of the file:
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@@
 		)
 	)
-	(label "ETH0.TRD3_N"
+	(label "TRD3_N"
 		(at 106.68 34.29 0)
 		(effects
@@
 		)
 	)
-	(label "ETH0.TRD2_N"
+	(label "TRD2_N"
 		(at 160.02 29.21 180)
 		(effects
@@
 		)
 	)
-	(label "ETH0.TRD1_P"
+	(label "TRD1_P"
 		(at 106.68 64.77 0)
 		(effects
@@
 		)
 	)
-	(label "ETH0.TRD1_N"
+	(label "TRD1_N"
 		(at 106.68 69.85 0)
 		(effects
@@
 		)
 	)
-	(label "ETH0.TRD0_N"
+	(label "TRD0_N"
 		(at 160.02 64.77 180)
 		(effects
@@
 		)
 	)
-	(label "ETH0.TRD3_P"
+	(label "TRD3_P"
 		(at 106.68 29.21 0)
 		(effects
@@
 		)
 	)
-	(label "ETH0.TRD0_P"
+	(label "TRD0_P"
 		(at 160.02 69.85 180)
 		(effects
@@
 		)
 	)
-	(label "ETH0.TRD2_P"
+	(label "TRD2_P"
 		(at 160.02 34.29 180)
 		(effects
@@
 		)
 	)
-	(hierarchical_label "ETH0{ETH0}"
+	(hierarchical_label "{ETH0}"
 		(shape bidirectional)
 		(at 20.32 99.06 270)
@@
 		)
 	)
-	(hierarchical_label "ETH0{ETH0}"
+	(hierarchical_label "{ETH0}"
 		(shape bidirectional)
 		(at 104.14 74.93 270)
@@
 		)
 	)
-	(hierarchical_label "ETH0{ETH0}"
+	(hierarchical_label "{ETH0}"
 		(shape bidirectional)
 		(at 162.56 74.93 270)
