File: hardware/ethernet.kicad_sch (KiCad schematic)
At the start: 7 parts, among them J9 THD-02-R, U1 TPD4EUSB30, U2 TPD4EUSB30, U3 MagJack-A70-112-331N126

Commit message: Small fixes
Parts:
- C1: Field4 Farnell -> (none); Field5 2611911 -> (none); Field6 RM EMK105 B7104KV-F -> (none); Field7 TAIYO YUDEN EUROPE GMBH -> (none); Field8 110091611 -> (none); MPN (none) -> GRM155R71C104KA88D; Manufacturer (none) -> Murata; Mouser (none) -> https://www.mouser.com/ProductDetail/81-GRM155R71C104KA88; Mouser PN (none) -> 81-GRM155R71C104KA88; Part Description 0.1uF 10% 16V Ceramic Capacitor X7R 0402 (1005 Metric) -> (none)
- J9: Field4 Toby -> (none); Field5 THD-02-R -> (none); Field6 151-604-425-761 -> (none); Field7 EDAC -> (none); Field8 UCON00791 -> (none); MPN (none) -> 61300421121; Manufacturer (none) -> Wurth Elektronik; Mouser (none) -> https://www.mouser.com/ProductDetail/710-61300421121; Mouser PN (none) -> 710-61300421121; Part Description PinHeader_2x02_P2.54mm_Vertical -> (none)
- R2, R3: Field4 Farnell -> (none); Field5 9239197 -> (none); Field6 RK73G1ETQTP4700D -> (none); Field7 KOA EUROPE GMBH -> (none); Field8 120887981 -> (none); MPN (none) -> RC0402FR-07470RL; Manufacturer (none) -> Yageo; Mouser (none) -> https://www.mouser.com/ProductDetail/603-RC0402FR-07470RL; Mouser PN (none) -> 603-RC0402FR-07470RL; Part Description Resistor 470R M1005 1% 63mW -> (none)
- U1, U2: Field4 Farnell -> (none); Field5 2335455 -> (none); Field6 CDDFN10-3324P-13 -> (none); Field7 Bourns -> (none); Field8 UDIO00346 -> (none); MPN (none) -> TPD4EUSB30DQAR; Manufacturer (none) -> Texas Instruments; Mouser (none) -> https://www.mouser.com/ProductDetail/595-TPD4EUSB30DQAR; Mouser PN (none) -> 595-TPD4EUSB30DQAR; Part Description Quad TVS diode for high speed signals (USB3, GigE etc.) -> (none)
- U3: Field5 TRJG0926HENL -> (none); Field6 TRJG0926HENL -> (none); Field7 Trxcon -> (none); Field8 UCON00900 -> (none); MPN (none) -> A70-112-331N126; Manufacturer (none) -> EDAC; Mouser (none) -> https://www.mouser.com/ProductDetail/587-A70-112-331N126; Mouser PN (none) -> 587-A70-112-331N126; Part Description Gigabit Ethernet Magjack -> (none)
Changed lines of the file:
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@@
 			)
 		)
-		(property "Datasheet" "https://p.globalsources.com/IMAGES/PDT/SPEC/690/K1160305690.pdf"
+		(property "Datasheet" "https://www.mouser.com/catalog/specsheets/EDAC_A70-112-331N126.pdf"
 			(at 80.01 106.68 0)
 			(hide yes)
@@
 			)
 		)
-		(property "Description" ""
+		(property "Description" "RJ45 MagJack 1000BASE-T, PoE-capable centre taps, LEDs"
 			(at 80.01 106.68 0)
 			(hide yes)
@@
 			)
 		)
-		(property "Field6" "TRJG0926HENL"
+		(property "Manufacturer" "EDAC"
 			(at 80.01 106.68 0)
 			(hide yes)
@@
 			)
 		)
-		(property "Field7" "Trxcon"
+		(property "MPN" "A70-112-331N126"
 			(at 80.01 106.68 0)
 			(hide yes)
@@
 			)
 		)
-		(property "Field8" "UCON00900"
+		(property "Mouser PN" "587-A70-112-331N126"
 			(at 80.01 106.68 0)
 			(hide yes)
@@
 			)
 		)
-		(property "Part Description" "Gigabit Ethernet Magjack"
-			(at 80.01 106.68 0)
-			(hide yes)
-			(show_name no)
-			(do_not_autoplace no)
-			(effects
-				(font
-					(size 1.27 1.27)
-				)
-			)
-		)
-		(property "Field5" "TRJG0926HENL"
+		(property "Mouser" "https://www.mouser.com/ProductDetail/587-A70-112-331N126"
 			(at 80.01 106.68 0)
 			(hide yes)
@@
 			)
 		)
-		(property "Datasheet" "https://fscdn.rohm.com/en/products/databook/datasheet/passive/resistor/chip_resistor/mcr-e.pdf"
+		(property "Datasheet" "https://yageogroup.com/content/datasheet/asset/file/PYU-RC_GROUP_51_ROHS_L"
 			(at 38.1 93.98 0)
 			(hide yes)
@@
 			)
 		)
-		(property "Description" ""
+		(property "Description" "RES 470R 1% 1/16W 0402"
 			(at 38.1 93.98 0)
 			(hide yes)
@@
 			)
 		)
-		(property "Field4" "Farnell"
+		(property "Manufacturer" "Yageo"
 			(at 38.1 93.98 0)
 			(hide yes)
@@
 			)
 		)
-		(property "Field5" "9239197"
+		(property "MPN" "RC0402FR-07470RL"
 			(at 38.1 93.98 0)
 			(hide yes)
@@
 			)
 		)
-		(property "Field7" "KOA EUROPE GMBH"
+		(property "Mouser PN" "603-RC0402FR-07470RL"
 			(at 38.1 93.98 0)
 			(hide yes)
@@
 			)
 		)
-		(property "Field6" "RK73G1ETQTP4700D         "
-			(at 38.1 93.98 0)
-			(hide yes)
-			(show_name no)
-			(do_not_autoplace no)
-			(effects
-				(font
-					(size 1.27 1.27)
-				)
-			)
-		)
-		(property "Field8" "120887981"
-			(at 38.1 93.98 0)
-			(hide yes)
-			(show_name no)
-			(do_not_autoplace no)
-			(effects
-				(font
-					(size 1.27 1.27)
-				)
-			)
-		)
-		(property "Part Description" "Resistor 470R M1005 1% 63mW"
+		(property "Mouser" "https://www.mouser.com/ProductDetail/603-RC0402FR-07470RL"
 			(at 38.1 93.98 0)
 			(hide yes)
@@
 			)
 		)
-		(property "Datasheet" "https://fscdn.rohm.com/en/products/databook/datasheet/passive/resistor/chip_resistor/mcr-e.pdf"
+		(property "Datasheet" "https://yageogroup.com/content/datasheet/asset/file/PYU-RC_GROUP_51_ROHS_L"
 			(at 38.1 88.9 0)
 			(hide yes)
@@
 			)
 		)
-		(property "Description" ""
+		(property "Description" "RES 470R 1% 1/16W 0402"
 			(at 38.1 88.9 0)
 			(hide yes)
@@
 			)
 		)
-		(property "Field4" "Farnell"
+		(property "Manufacturer" "Yageo"
 			(at 38.1 88.9 0)
 			(hide yes)
@@
 			)
 		)
-		(property "Field5" "9239197"
+		(property "MPN" "RC0402FR-07470RL"
 			(at 38.1 88.9 0)
 			(hide yes)
@@
 			)
 		)
-		(property "Field7" "KOA EUROPE GMBH"
+		(property "Mouser PN" "603-RC0402FR-07470RL"
 			(at 38.1 88.9 0)
 			(hide yes)
@@
 			)
 		)
-		(property "Field6" "RK73G1ETQTP4700D         "
-			(at 38.1 88.9 0)
-			(hide yes)
-			(show_name no)
-			(do_not_autoplace no)
-			(effects
-				(font
-					(size 1.27 1.27)
-				)
-			)
-		)
-		(property "Field8" "120887981"
-			(at 38.1 88.9 0)
-			(hide yes)
-			(show_name no)
-			(do_not_autoplace no)
-			(effects
-				(font
-					(size 1.27 1.27)
-				)
-			)
-		)
-		(property "Part Description" "Resistor 470R M1005 1% 63mW"
+		(property "Mouser" "https://www.mouser.com/ProductDetail/603-RC0402FR-07470RL"
 			(at 38.1 88.9 0)
 			(hide yes)
@@
 			)
 		)
-		(property "Datasheet" "http://www.ti.com/lit/ds/symlink/tpd2eusb30a.pdf"
+		(property "Datasheet" "https://www.ti.com/lit/ds/symlink/tpd4eusb30.pdf"
 			(at 133.35 31.75 0)
 			(hide yes)
@@
 			)
 		)
-		(property "Description" ""
+		(property "Description" "ESD array 4-ch 0.8pF USON-10"
 			(at 133.35 31.75 0)
 			(hide yes)
@@
 			)
 		)
-		(property "Field4" "Farnell"
+		(property "Manufacturer" "Texas Instruments"
 			(at 133.35 31.75 0)
 			(hide yes)
@@
 			)
 		)
-		(property "Field5" "2335455"
+		(property "MPN" "TPD4EUSB30DQAR"
 			(at 133.35 31.75 0)
 			(hide yes)
@@
 			)
 		)
-		(property "Field6" "CDDFN10-3324P-13"
+		(property "Mouser PN" "595-TPD4EUSB30DQAR"
 			(at 133.35 31.75 0)
 			(hide yes)
@@
 			)
 		)
-		(property "Field7" "Bourns"
-			(at 133.35 31.75 0)
-			(hide yes)
-			(show_name no)
-			(do_not_autoplace no)
-			(effects
-				(font
-					(size 1.27 1.27)
-				)
-			)
-		)
-		(property "Field8" "UDIO00346"
-			(at 133.35 31.75 0)
-			(hide yes)
-			(show_name no)
-			(do_not_autoplace no)
-			(effects
-				(font
-					(size 1.27 1.27)
-				)
-			)
-		)
-		(property "Part Description" "Quad TVS diode for high speed signals (USB3, GigE etc.)"
+		(property "Mouser" "https://www.mouser.com/ProductDetail/595-TPD4EUSB30DQAR"
 			(at 133.35 31.75 0)
 			(hide yes)
@@
 			)
 		)
-		(property "Datasheet" "https://search.murata.co.jp/Ceramy/image/img/A01X/G101/ENG/GRM155R71C104KA88-01.pdf"
+		(property "Datasheet" "https://pim.murata.com/asset/pim4/ceramicCapacitorSMD/GRM155R71C104KA88-01A-EN_PDF_CERAMICCAPACITORSMD"
 			(at 46.99 102.87 0)
 			(hide yes)
@@
 			)
 		)
-		(property "Description" ""
+		(property "Description" "CAP CER 100nF 16V X7R 10% 0402"
 			(at 46.99 102.87 0)
 			(hide yes)
@@
 			)
 		)
-		(property "Field4" "Farnell"
+		(property "Manufacturer" "Murata"
 			(at 46.99 102.87 0)
 			(hide yes)
@@
 			)
 		)
-		(property "Field5" "2611911"
+		(property "MPN" "GRM155R71C104KA88D"
 			(at 46.99 102.87 0)
 			(hide yes)
@@
 			)
 		)
-		(property "Field6" "RM EMK105 B7104KV-F"
+		(property "Mouser PN" "81-GRM155R71C104KA88"
 			(at 46.99 102.87 0)
 			(hide yes)
@@
 			)
 		)
-		(property "Field7" "TAIYO YUDEN EUROPE GMBH"
-			(at 46.99 102.87 0)
-			(hide yes)
-			(show_name no)
-			(do_not_autoplace no)
-			(effects
-				(font
-					(size 1.27 1.27)
-				)
-			)
-		)
-		(property "Part Description" "	0.1uF 10% 16V Ceramic Capacitor X7R 0402 (1005 Metric)"
-			(at 46.99 102.87 0)
-			(hide yes)
-			(show_name no)
-			(do_not_autoplace no)
-			(effects
-				(font
-					(size 1.27 1.27)
-				)
-			)
-		)
-		(property "Field8" "110091611"
+		(property "Mouser" "https://www.mouser.com/ProductDetail/81-GRM155R71C104KA88"
 			(at 46.99 102.87 0)
 			(hide yes)
@@
 			)
 		)
-		(property "Datasheet" "http://www.ti.com/lit/ds/symlink/tpd2eusb30a.pdf"
+		(property "Datasheet" "https://www.ti.com/lit/ds/symlink/tpd4eusb30.pdf"
 			(at 133.35 67.31 0)
 			(hide yes)
@@
 			)
 		)
-		(property "Description" ""
+		(property "Description" "ESD array 4-ch 0.8pF USON-10"
 			(at 133.35 67.31 0)
 			(hide yes)
@@
 			)
 		)
-		(property "Field4" "Farnell"
+		(property "Manufacturer" "Texas Instruments"
 			(at 133.35 67.31 0)
 			(hide yes)
@@
 			)
 		)
-		(property "Field5" "2335455"
+		(property "MPN" "TPD4EUSB30DQAR"
 			(at 133.35 67.31 0)
 			(hide yes)
@@
 			)
 		)
-		(property "Field6" "CDDFN10-3324P-13"
+		(property "Mouser PN" "595-TPD4EUSB30DQAR"
 			(at 133.35 67.31 0)
 			(hide yes)
@@
 			)
 		)
-		(property "Field7" "Bourns"
-			(at 133.35 67.31 0)
-			(hide yes)
-			(show_name no)
-			(do_not_autoplace no)
-			(effects
-				(font
-					(size 1.27 1.27)
-				)
-			)
-		)
-		(property "Field8" "UDIO00346"
-			(at 133.35 67.31 0)
-			(hide yes)
-			(show_name no)
-			(do_not_autoplace no)
-			(effects
-				(font
-					(size 1.27 1.27)
-				)
-			)
-		)
-		(property "Part Description" "Quad TVS diode for high speed signals (USB3, GigE etc.)"
+		(property "Mouser" "https://www.mouser.com/ProductDetail/595-TPD4EUSB30DQAR"
 			(at 133.35 67.31 0)
 			(hide yes)
@@
 			)
 		)
-		(property "Datasheet" "https://www.toby.co.uk/uploads/publications/1673.pdf"
+		(property "Datasheet" "https://www.we-online.com/components/products/datasheet/61300421121.pdf"
 			(at 187.96 25.4 0)
 			(hide yes)
@@
 			)
 		)
-		(property "Description" ""
+		(property "Description" "CONN HDR 2x2 2.54mm vertical THT"
 			(at 187.96 25.4 0)
 			(hide yes)
@@
 			)
 		)
-		(property "Field4" "Toby"
+		(property "Manufacturer" "Wurth Elektronik"
 			(at 187.96 25.4 0)
 			(hide yes)
@@
 			)
 		)
-		(property "Field5" "THD-02-R"
+		(property "MPN" "61300421121"
 			(at 187.96 25.4 0)
 			(hide yes)
@@
 			)
 		)
-		(property "Field6" "151-604-425-761"
+		(property "Mouser PN" "710-61300421121"
 			(at 187.96 25.4 0)
 			(hide yes)
@@
 			)
 		)
-		(property "Field7" "EDAC"
+		(property "Mouser" "https://www.mouser.com/ProductDetail/710-61300421121"
 			(at 187.96 25.4 0)
 			(hide yes)
-			(show_name no)
-			(do_not_autoplace no)
-			(effects
-				(font
-					(size 1.27 1.27)
-				)
-			)
-		)
-		(property "Field8" "UCON00791"
-			(at 187.96 25.4 0)
-			(hide yes)
-			(show_name no)
-			(do_not_autoplace no)
-			(effects
-				(font
-					(size 1.27 1.27)
-				)
-			)
-		)
-		(property "Part Description" "PinHeader_2x02_P2.54mm_Vertical"
-			(at 187.96 25.4 0)
-			(hide yes)

Commit message: Add rudimenatry poe module
Parts:
- removed J9: THD-02-R, Connector_PinHeader_2.54mm:PinHeader_2x02_P2.54mm_Vertical, symbol Connector_Generic:Conn_02x02_Odd_Even
Other:
- note removed: "POE Header"

Commit message: Add PoE circuit
Connections:
- net TR0_TAP renamed VC1
- net TR1_TAP renamed VC2
- net TR2_TAP renamed VC3
- net TR3_TAP renamed VC4
Changed lines of the file:
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@@
+	)
+	(bus_entry
+		(at 22.86 78.74)
+		(size -2.54 2.54)
+		(stroke
+			(width 0)
+			(type default)
+		)
 	)
 	(bus_entry
@@
 	(bus_entry
 		(at 22.86 88.9)
+		(size -2.54 2.54)
+		(stroke
+			(width 0)
+			(type default)
+		)
+	)
+	(bus_entry
+		(at 22.86 81.28)
 		(size -2.54 2.54)
 		(stroke
@@
 	)
 	(bus_entry
+		(at 22.86 73.66)
+		(size -2.54 2.54)
+		(stroke
+			(width 0)
+			(type default)
+		)
+	)
+	(bus_entry
 		(at 104.14 31.75)
 		(size 2.54 -2.54)
@@
 	)
 	(bus_entry
+		(at 22.86 76.2)
+		(size -2.54 2.54)
+		(stroke
+			(width 0)
+			(type default)
+		)
+	)
+	(bus_entry
 		(at 22.86 68.58)
 		(size -2.54 2.54)
@@
 		)
 	)
-	(label "TR0_TAP"
+	(label "VC1"
 		(at 22.86 73.66 0)
 		(effects
@@
 		)
 	)
-	(label "TR2_TAP"
+	(label "VC3"
 		(at 22.86 78.74 0)
 		(effects
@@
 		)
 	)
-	(label "TR1_TAP"
+	(label "VC2"
 		(at 22.86 76.2 0)
 		(effects
@@
 		)
 	)
-	(label "TR3_TAP"
+	(label "VC4"
 		(at 22.86 81.28 0)
 		(effects
