File: hardware/i2c_peripherals.kicad_sch (KiCad schematic)
At the start: 8 parts, among them IC1 BMI270, IC2 SHT45-AD1F-R2, J1 Conn_01x04_Pin

Commit message: Assign footprints to all parts
Connectors get footprints for the chosen hardware: JST GH for the ESC
and pressure-sensor cables, XT30 for the battery and the GCT USB4105
for the service port. The core regulator inductor and the SWD
connector use the footprints from Raspberry Pi's RP2350A minimal
design, which is MIT-licensed and credited in NOTICE.md. Every symbol
pin now has a matching pad.

Co-Authored-By: Claude Opus 5.5 <noreply@anthropic.com>
Parts:
- IC1: footprint BMI270 -> BMI270:BMI270
- IC2: footprint SON80P150X150X59-5N -> SHT45:SON80P150X150X59-5N
- J1: footprint Connector:Tag-Connect_TC2030-IDC-FP_2x03_P1.27mm_Vertical -> Connector_JST:JST_GH_SM04B-GHS-TB_1x04-1MP_P1.25mm_Horizontal
Changed lines of the file:
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@@
 			)
 		)
-		(property "Footprint" "Connector:Tag-Connect_TC2030-IDC-FP_2x03_P1.27mm_Vertical"
+		(property "Footprint" "Connector_JST:JST_GH_SM04B-GHS-TB_1x04-1MP_P1.25mm_Horizontal"
 			(at 66.04 27.94 0)
 			(hide yes)
@@
 			)
 		)
-		(property "Footprint" "BMI270"
+		(property "Footprint" "BMI270:BMI270"
 			(at -18.72 83.82 0)
 			(hide yes)
@@
 			)
 		)
-		(property "Footprint" "SON80P150X150X59-5N"
+		(property "Footprint" "SHT45:SON80P150X150X59-5N"
 			(at 146.05 157.15 0)
 			(hide yes)
