File: hardware/i2c_peripherals.kicad_sch (KiCad schematic)
At the start: 10 parts, among them IC1 BMI270, IC2 SHT45-AD1F-R2, J1 Conn_01x04_Pin, U10 WSEN-PADS_2511020213301

Commit message: Add LCSC part numbers and links, fix J7 part number
- Every part found on LCSC gets an "LCSC PN" (C-number) and an "LCSC" product
  link field, in the schematic and on the PCB footprints. Exact matches where
  LCSC lists the part; equivalents with the same specs where it does not or
  has no stock (C46, C26/C28/C30/C33/C34/C40, C29, C31, R6/R7, R21, R24,
  J3/J4, J7/J9/J13). Left empty: IC3, IC5 (not on LCSC), IC10, IC12
  (JLCPCB-only listings).
- J7: the MPN 61301421121 is a 2.54 mm header, but the footprint is 1.27 mm.
  Now Wurth 62201421121 (WR-PHD 1.27 mm 2x7) with matching description,
  datasheet and Mouser fields.
- Interactive HTML BOM in hardware/bom; KiCad project file re-saved.

Co-Authored-By: Claude Opus 5.5 <noreply@anthropic.com>
Claude-Session: https://claude.ai/code/session_01AhLYztcZikG9g81njGtEr1
Parts:
- C2, C3, C38, C4: LCSC (none) -> https://www.lcsc.com/product-detail/C71629.html; LCSC PN (none) -> C71629
- IC1, IC2: LCSC (none) -> https://www.lcsc.com/product-detail/C90627.html; LCSC PN (none) -> C90627
- J1: LCSC (none) -> https://www.lcsc.com/product-detail/C189895.html; LCSC PN (none) -> C189895
- R4, R5: LCSC (none) -> https://www.lcsc.com/product-detail/C114762.html; LCSC PN (none) -> C114762
Changed lines of the file:
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@@
+			)
+		)
+		(property "LCSC PN" "C114762"
+			(at 30.48 33.02 0)
+			(hide yes)
+			(show_name no)
+			(do_not_autoplace no)
+			(effects
+				(font
+					(size 1.27 1.27)
+				)
+			)
+		)
+		(property "LCSC" "https://www.lcsc.com/product-detail/C114762.html"
+			(at 30.48 33.02 0)
+			(hide yes)
+			(show_name no)
+			(do_not_autoplace no)
+			(effects
+				(font
+					(size 1.27 1.27)
+				)
 			)
 		)
@@
 		)
 		(property "Mouser" "https://www.mouser.com/ProductDetail/81-GRM155R71C104KA88"
+			(at 142.2513 46.9724 0)
+			(hide yes)
+			(show_name no)
+			(do_not_autoplace no)
+			(effects
+				(font
+					(size 1.27 1.27)
+				)
+			)
+		)
+		(property "LCSC PN" "C71629"
+			(at 142.2513 46.9724 0)
+			(hide yes)
+			(show_name no)
+			(do_not_autoplace no)
+			(effects
+				(font
+					(size 1.27 1.27)
+				)
+			)
+		)
+		(property "LCSC" "https://www.lcsc.com/product-detail/C71629.html"
 			(at 142.2513 46.9724 0)
 			(hide yes)
@@
 			)
 		)
+		(property "LCSC PN" "C189895"
+			(at 68.58 35.56 0)
+			(hide yes)
+			(show_name no)
+			(do_not_autoplace no)
+			(effects
+				(font
+					(size 1.27 1.27)
+				)
+			)
+		)
+		(property "LCSC" "https://www.lcsc.com/product-detail/C189895.html"
+			(at 68.58 35.56 0)
+			(hide yes)
+			(show_name no)
+			(do_not_autoplace no)
+			(effects
+				(font
+					(size 1.27 1.27)
+				)
+			)
+		)
 		(pin "4"
 		)
@@
 		)
 		(property "Mouser" "https://www.mouser.com/ProductDetail/81-GRM155R71C104KA88"
+			(at 31.75 124.46 0)
+			(hide yes)
+			(show_name no)
+			(do_not_autoplace no)
+			(effects
+				(font
+					(size 1.27 1.27)
+				)
+			)
+		)
+		(property "LCSC PN" "C71629"
+			(at 31.75 124.46 0)
+			(hide yes)
+			(show_name no)
+			(do_not_autoplace no)
+			(effects
+				(font
+					(size 1.27 1.27)
+				)
+			)
+		)
+		(property "LCSC" "https://www.lcsc.com/product-detail/C71629.html"
 			(at 31.75 124.46 0)
 			(hide yes)
@@
 			)
 		)
+		(property "LCSC PN" "C71629"
+			(at 236.22 43.18 0)
+			(hide yes)
+			(show_name no)
+			(do_not_autoplace no)
+			(effects
+				(font
+					(size 1.27 1.27)
+				)
+			)
+		)
+		(property "LCSC" "https://www.lcsc.com/product-detail/C71629.html"
+			(at 236.22 43.18 0)
+			(hide yes)
+			(show_name no)
+			(do_not_autoplace no)
+			(effects
+				(font
+					(size 1.27 1.27)
+				)
+			)
+		)
 		(pin "1"
 		)
@@
 		)
 		(property "Mouser" "https://www.mouser.com/ProductDetail/81-GRM155R71C104KA88"
+			(at 62.23 124.46 0)
+			(hide yes)
+			(show_name no)
+			(do_not_autoplace no)
+			(effects
+				(font
+					(size 1.27 1.27)
+				)
+			)
+		)
+		(property "LCSC PN" "C71629"
+			(at 62.23 124.46 0)
+			(hide yes)
+			(show_name no)
+			(do_not_autoplace no)
+			(effects
+				(font
+					(size 1.27 1.27)
+				)
+			)
+		)
+		(property "LCSC" "https://www.lcsc.com/product-detail/C71629.html"
 			(at 62.23 124.46 0)
 			(hide yes)
@@
 			)
 		)
+		(property "LCSC PN" "C90627"
+			(at 69.85 85.09 0)
+			(hide yes)
+			(show_name no)
+			(do_not_autoplace no)
+			(effects
+				(font
+					(size 1.27 1.27)
+				)
+			)
+		)
+		(property "LCSC" "https://www.lcsc.com/product-detail/C90627.html"
+			(at 69.85 85.09 0)
+			(hide yes)
+			(show_name no)
+			(do_not_autoplace no)
+			(effects
+				(font
+					(size 1.27 1.27)
+				)
+			)
+		)
 		(pin "13"
 		)
@@
 			)
 		)
+		(property "LCSC PN" "C90627"
+			(at 106.6913 38.0824 0)
+			(hide yes)
+			(show_name no)
+			(do_not_autoplace no)
+			(effects
+				(font
+					(size 1.27 1.27)
+				)
+			)
+		)
+		(property "LCSC" "https://www.lcsc.com/product-detail/C90627.html"
+			(at 106.6913 38.0824 0)
+			(hide yes)
+			(show_name no)
+			(do_not_autoplace no)
+			(effects
+				(font
+					(size 1.27 1.27)
+				)
+			)
+		)
 		(pin "4"
 		)
@@
 			(at 40.64 33.02 0)
 			(hide yes)
+			(show_name no)
+			(do_not_autoplace no)
+			(effects
+				(font
+					(size 1.27 1.27)
+				)
+			)
+		)
+		(property "LCSC PN" "C114762"
+			(at 40.64 33.02 0)
+			(hide yes)
+			(show_name no)
+			(do_not_autoplace no)
+			(effects
+				(font
+					(size 1.27 1.27)
+				)
+			)
+		)
+		(property "LCSC" "https://www.lcsc.com/product-detail/C114762.html"
+			(at 40.64 33.02 0)
+			(hide yes)
