File: hardware/rp2354a.kicad_sch (KiCad schematic)
At the start: 25 parts, among them J2 SM03B-SRSS-TB, J3 AM32_1, J4 AM32_2, U4 RP2354A

Commit message: Fix schematic connectivity and add flashing access
The camera and Ethernet buses now connect across sheets: they use
unnamed bus groups so the member nets keep their names. Ethernet pair 2
negative is no longer tied to GND.

The RP2354A core supply reaches the regulator output, and a 12 MHz
crystal drives XIN/XOUT, which USB and the USB bootloader need. The
CM5 gets GPIO_VREF on 3.3 V, the IO Board's boot and EEPROM jumper
header, and a data-only USB-C port with 5.1 kOhm CC resistors for
flashing the eMMC.

Co-Authored-By: Claude Opus 5.5 <noreply@anthropic.com>
Parts:
- added C18, C19: 15pF, Capacitor_SMD:C_0402_1005Metric, symbol Device:C
- added R10: 1kR, Resistor_SMD:R_0402_1005Metric, symbol Device:R
- added Y1: ABM8-272-T3, ABM8272T3, symbol ABM8-272-T3:ABM8-272-T3
Connections:
- net +1.1V: now also U4.23 (DVDD), U4.39 (DVDD), U4.6 (DVDD)
- net GND: now also C18.2, C19.2, Y1.2 (GND_1), Y1.4 (GND_2)
- net XIN: now reaches U4.21 (XIN)
- net XIN: now also C18.1, Y1.1 (CRYSTAL_1)
- net XOUT: now reaches U4.22 (XOUT)
- net XOUT: now also R10.2
- new net: C19.1, R10.1, Y1.3 (CRYSTAL_2)
- no-connect marks 7 -> 5
Other:
- note added: "Crystal"
- note added: "Note: Required for USB or UART"
- moved on the sheet: C14, C15, L1

Commit message: Assign footprints to all parts
Connectors get footprints for the chosen hardware: JST GH for the ESC
and pressure-sensor cables, XT30 for the battery and the GCT USB4105
for the service port. The core regulator inductor and the SWD
connector use the footprints from Raspberry Pi's RP2350A minimal
design, which is MIT-licensed and credited in NOTICE.md. Every symbol
pin now has a matching pad.

Co-Authored-By: Claude Opus 5.5 <noreply@anthropic.com>
Parts:
- J2: footprint (none) -> RP2350_Minimal:jst_sm03b-srss-tb-lf--sn-
- J3, J4: footprint (none) -> Connector_JST:JST_GH_SM05B-GHS-TB_1x05-1MP_P1.25mm_Horizontal
- L1: footprint Package_DFN_QFN:QFN-60-1EP_7x7mm_P0.4mm_EP3.4x3.4mm -> RP2350_Minimal:abracon_aota-b201610s3r3-101-t
- Y1: footprint ABM8272T3 -> ABM8-272-T3:ABM8272T3
Changed lines of the file:
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@@
 			)
 		)
-		(property "Footprint" "Package_DFN_QFN:QFN-60-1EP_7x7mm_P0.4mm_EP3.4x3.4mm"
+		(property "Footprint" "RP2350_Minimal:abracon_aota-b201610s3r3-101-t"
 			(at 166.37 36.83 0)
 			(hide yes)
@@
 			)
 		)
-		(property "Footprint" ""
+		(property "Footprint" "RP2350_Minimal:jst_sm03b-srss-tb-lf--sn-"
 			(at 58.42 172.72 0)
 			(hide yes)
@@
 			)
 		)
-		(property "Footprint" ""
+		(property "Footprint" "Connector_JST:JST_GH_SM05B-GHS-TB_1x05-1MP_P1.25mm_Horizontal"
 			(at 137.16 116.84 0)
 			(hide yes)
@@
 			)
 		)
-		(property "Footprint" "ABM8272T3"
+		(property "Footprint" "ABM8-272-T3:ABM8272T3"
 			(at 204.47 168.58 0)
 			(hide yes)
@@
 			)
 		)
-		(property "Footprint" ""
+		(property "Footprint" "Connector_JST:JST_GH_SM05B-GHS-TB_1x05-1MP_P1.25mm_Horizontal"
 			(at 137.16 147.32 0)
 			(hide yes)
