File: hardware/rp2354a.kicad_sch (KiCad schematic)
At the start: 29 parts, among them J2 SM03B-SRSS-TB, J3 AM32_1, J4 AM32_2, U4 RP2354A, Y1 ABM8-272-T3

Commit message: Small fixes
Parts:
- added R16, R17: 33R, Resistor_SMD:R_0402_1005Metric, symbol Device:R
- C10, C11, C12, C13, C16, C5, C6, C7, C8, C9: Field4 Farnell -> (none); Field5 2611911 -> (none); Field6 RM EMK105 B7104KV-F -> (none); Field7 TAIYO YUDEN EUROPE GMBH -> (none); Field8 110091611 -> (none); MPN (none) -> GRM155R71C104KA88D; Manufacturer (none) -> Murata; Mouser (none) -> https://www.mouser.com/ProductDetail/81-GRM155R71C104KA88; Mouser PN (none) -> 81-GRM155R71C104KA88; Part Description 0.1uF 10% 16V Ceramic Capacitor X7R 0402 (1005 Metric) -> (none)
- C14, C15, C17: Field4 Farnell -> (none); Field5 2611911 -> (none); Field6 RM EMK105 B7104KV-F -> (none); Field7 TAIYO YUDEN EUROPE GMBH -> (none); Field8 110091611 -> (none); MPN (none) -> GRM155R60J475ME47D; Manufacturer (none) -> Murata; Mouser (none) -> https://www.mouser.com/ProductDetail/81-GRM155R60J475ME7D; Mouser PN (none) -> 81-GRM155R60J475ME7D; Part Description 0.1uF 10% 16V Ceramic Capacitor X7R 0402 (1005 Metric) -> (none)
- C18, C19: Field4 Farnell -> (none); Field5 2611911 -> (none); Field6 RM EMK105 B7104KV-F -> (none); Field7 TAIYO YUDEN EUROPE GMBH -> (none); Field8 110091611 -> (none); MPN (none) -> GRM1555C1H150JA01D; Manufacturer (none) -> Murata; Mouser (none) -> https://www.mouser.com/ProductDetail/81-GRM1555C1H150JA1D; Mouser PN (none) -> 81-GRM1555C1H150JA1D; Part Description 0.1uF 10% 16V Ceramic Capacitor X7R 0402 (1005 Metric) -> (none)
- J2: MPN (none) -> SM03B-SRSS-TB(LF)(SN); Manufacturer (none) -> JST; Mouser (none) -> https://www.mouser.com/ProductDetail/306-SM03BSRSSTBLFSNP; Mouser PN (none) -> 306-SM03BSRSSTBLFSNP
- J3, J4: MPN (none) -> SM05B-GHS-TB(LF)(SN); Manufacturer (none) -> JST; Mouser (none) -> https://www.mouser.com/ProductDetail/306-SM05BGHSTBLFSN; Mouser PN (none) -> 306-SM05BGHSTBLFSN
- L1: MPN (none) -> AOTA-B201610S3R3-101-T; Manufacturer (none) -> Abracon; Mouser (none) -> https://www.mouser.com/ProductDetail/815-AB201610S3R3101T; Mouser PN (none) -> 815-AB201610S3R3101T; Note (none) -> Required part (RP2350 hardware design guide), do not substi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
- R10, R12: MPN (none) -> RC0402FR-071KL; Manufacturer (none) -> Yageo; Mouser (none) -> https://www.mouser.com/ProductDetail/603-RC0402FR-071KL; Mouser PN (none) -> 603-RC0402FR-071KL
- R11: MPN (none) -> RC0402FR-074K7L; Manufacturer (none) -> Yageo; Mouser (none) -> https://www.mouser.com/ProductDetail/603-RC0402FR-074K7L; Mouser PN (none) -> 603-RC0402FR-074K7L
- R13: MPN (none) -> RC0402FR-0710KL; Manufacturer (none) -> Yageo; Mouser (none) -> https://www.mouser.com/ProductDetail/603-RC0402FR-0710KL; Mouser PN (none) -> 603-RC0402FR-0710KL
- R6, R7: MPN (none) -> RC0402FR-0727RL; Manufacturer (none) -> Yageo; Mouser (none) -> https://www.mouser.com/ProductDetail/603-RC0402FR-0727RL; Mouser PN (none) -> 603-RC0402FR-0727RL
- R8: MPN (none) -> RC0402FR-0733RL; Manufacturer (none) -> Yageo; Mouser (none) -> https://www.mouser.com/ProductDetail/603-RC0402FR-0733RL; Mouser PN (none) -> 603-RC0402FR-0733RL
- R9: MPN (none) -> RC0402FR-07330RL; Manufacturer (none) -> Yageo; Mouser (none) -> https://www.mouser.com/ProductDetail/603-RC0402FR-07330RL; Mouser PN (none) -> 603-RC0402FR-07330RL
- U4: MPN (none) -> SC1511-A4; Manufacturer (none) -> Raspberry Pi; Mouser (none) -> https://www.mouser.com/ProductDetail/Raspberry-Pi/SC1511-A4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; Mouser PN (none) -> 358-SC1511; Note (none) -> Mouser sells full 500-pc reels only; for prototypes buy cut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
- Y1: MPN (none) -> ABM8-272-T3; Manufacturer (none) -> Abracon; Manufacturer_Name ABRACON -> (none); Manufacturer_Part_Number ABM8-272-T3 -> (none); Mouser (none) -> https://www.mouser.com/ProductDetail/815-ABM8-272-T3; Mouser PN (none) -> 815-ABM8-272-T3; Mouser Part Number 815-ABM8-272-T3 -> (none); Mouser Price/Stock https://www.mouser.co.uk/ProductDetail/ABRACON/ABM8-272-T3?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 -> (none)
Connections:
- net +1.1V: now also L1.1; no longer L1.2
- net GND: now also J3.5 (Pin_5), J4.5 (Pin_5); no longer J3.1 (Pin_1), J4.1 (Pin_1)
- net VREG_LX: now also L1.2; no longer L1.1
- net at J2.1 (Pin_1), U4.24 (SWCLK): now also R16.1
- net at J2.3 (Pin_3), U4.25 (SWDIO): now also R17.1
- net at J3.2 (Pin_2): now also U4.10 (GPIO7); no longer U4.13 (GPIO9)
- net at J3.4 (Pin_4): now also U4.13 (GPIO9); no longer U4.10 (GPIO7)
- net at U4.9 (GPIO6): now also J3.1 (Pin_1); no longer J3.5 (Pin_5)
- net at J4.2 (Pin_2): now also U4.31 (GPIO19); no longer U4.33 (GPIO21)
- net at J4.4 (Pin_4): now also U4.33 (GPIO21); no longer U4.31 (GPIO19)
- net at U4.29 (GPIO18): now also J4.1 (Pin_1); no longer J4.5 (Pin_5)
- new net RP2354_SWCLK: R16.2
- new net RP2354_SWDIO: R17.2
Other:
- moved on the sheet: J2, J3, J4, L1

Commit message: Update sensor connection, add 3d files
Connections:
- net I2C0_SCL: now reaches U4.5 (GPIO3)
- net I2C0_SDA: now reaches U4.7 (GPIO4)
Changed lines of the file:
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@@
+	(wire
+		(pts
+			(xy 121.92 104.14) (xy 124.46 104.14)
+		)
+		(stroke
+			(width 0)
+			(type default)
+		)
+	)
 	(wire
 		(pts
@@
 		(pts
 			(xy 58.42 27.94) (xy 58.42 30.48)
+		)
+		(stroke
+			(width 0)
+			(type default)
+		)
+	)
+	(wire
+		(pts
+			(xy 121.92 106.68) (xy 124.46 106.68)
 		)
 		(stroke
@@
 		)
 	)
+	(hierarchical_label "I2C0_SCL"
+		(shape output)
+		(at 124.46 104.14 0)
+		(effects
+			(font
+				(size 1.27 1.27)
+			)
+			(justify left)
+		)
+	)
 	(hierarchical_label "USB_D-"
 		(shape bidirectional)
@@
 		)
 	)
+	(hierarchical_label "I2C0_SDA"
+		(shape bidirectional)
+		(at 124.46 106.68 0)
+		(effects
+			(font
+				(size 1.27 1.27)
+			)
+			(justify left)
+		)
+	)
