File: hardware/rp2354a.kicad_sch (KiCad schematic)
At the start: 32 parts, among them IC4 RP2354A, J13 Conn_02x06_Odd_Even, J2 SM03B-SRSS-TB, J3 AM32_1, J4 AM32_2, Y1 ABM8-272-T3

Commit message: Redo the PCB layout (rev 3): 70 x 109.2 mm, connectors on one side, 45° routing
- All connectors on the top: cameras, USB-C and the magnet switch along the
  top edge, the rest at the bottom around the RJ45, which moves towards the
  centre line; C20 near the centre for the tube radius
- Every part except the PoE module IC5 on the top (reflow one side)
- 45-degree routing only, chamfers at least 1.5 x width, traces bundled to
  keep the planes whole
- Small SHT45 tongue with its bypass cap beside it; planes cut out under L2
  with nothing under it; copper 3.4 mm from the CM5 mounting holes
- Charger and RP2354A regulator laid out per their datasheets
- J3/J4 vertical JST GH (BM05B-GHS-TBT); J8 VBUS label restored
- Edge clearance 0.3 mm, netclass patterns follow the current net names,
  hand-soldered THT GND pins get one thermal spoke
- User.Comments fab/assembly notes and README PCB section updated for rev 3

Co-Authored-By: Claude Opus 5.5 <noreply@anthropic.com>
Parts:
- J3, J4: footprint Connector_JST:JST_GH_SM05B-GHS-TB_1x05-1MP_P1.25mm_Horizontal -> Connector_JST:JST_GH_BM05B-GHS-TBT_1x05-1MP_P1.25mm_Vertical; MPN SM05B-GHS-TB(LF)(SN) -> BM05B-GHS-TBT(LF)(SN); Mouser PN 306-SM05BGHSTBLFSN -> (none)
Changed lines of the file:
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@@
 			)
 		)
-		(property "Footprint" "Connector_JST:JST_GH_SM05B-GHS-TB_1x05-1MP_P1.25mm_Horizontal"
+		(property "Footprint" "Connector_JST:JST_GH_BM05B-GHS-TBT_1x05-1MP_P1.25mm_Vertical"
 			(at 142.24 116.84 0)
 			(hide yes)
@@
 			)
 		)
-		(property "Description" "CONN JST GH 5P 1.25mm R/A SMD"
+		(property "Description" "CONN JST GH 5P 1.25mm vertical SMD"
 			(at 142.24 116.84 0)
 			(hide yes)
@@
 			)
 		)
-		(property "MPN" "SM05B-GHS-TB(LF)(SN)"
+		(property "MPN" "BM05B-GHS-TBT(LF)(SN)"
 			(at 142.24 116.84 0)
 			(hide yes)
@@
 			)
 		)
-		(property "Mouser PN" "306-SM05BGHSTBLFSN"
+		(property "Mouser PN" ""
 			(at 142.24 116.84 0)
 			(hide yes)
@@
 			)
 		)
-		(property "Footprint" "Connector_JST:JST_GH_SM05B-GHS-TB_1x05-1MP_P1.25mm_Horizontal"
+		(property "Footprint" "Connector_JST:JST_GH_BM05B-GHS-TBT_1x05-1MP_P1.25mm_Vertical"
 			(at 143.51 147.32 0)
 			(hide yes)
@@
 			)
 		)
-		(property "Description" "CONN JST GH 5P 1.25mm R/A SMD"
+		(property "Description" "CONN JST GH 5P 1.25mm vertical SMD"
 			(at 143.51 147.32 0)
 			(hide yes)
@@
 			)
 		)
-		(property "MPN" "SM05B-GHS-TB(LF)(SN)"
+		(property "MPN" "BM05B-GHS-TBT(LF)(SN)"
 			(at 143.51 147.32 0)
 			(hide yes)
@@
 			)
 		)
-		(property "Mouser PN" "306-SM05BGHSTBLFSN"
+		(property "Mouser PN" ""
 			(at 143.51 147.32 0)
 			(hide yes)

Commit message: Add LCSC part numbers and links, fix J7 part number
- Every part found on LCSC gets an "LCSC PN" (C-number) and an "LCSC" product
  link field, in the schematic and on the PCB footprints. Exact matches where
  LCSC lists the part; equivalents with the same specs where it does not or
  has no stock (C46, C26/C28/C30/C33/C34/C40, C29, C31, R6/R7, R21, R24,
  J3/J4, J7/J9/J13). Left empty: IC3, IC5 (not on LCSC), IC10, IC12
  (JLCPCB-only listings).
- J7: the MPN 61301421121 is a 2.54 mm header, but the footprint is 1.27 mm.
  Now Wurth 62201421121 (WR-PHD 1.27 mm 2x7) with matching description,
  datasheet and Mouser fields.
- Interactive HTML BOM in hardware/bom; KiCad project file re-saved.

Co-Authored-By: Claude Opus 5.5 <noreply@anthropic.com>
Claude-Session: https://claude.ai/code/session_01AhLYztcZikG9g81njGtEr1
Parts:
- C10, C11, C12, C13, C16, C5, C6, C7, C8, C9: LCSC (none) -> https://www.lcsc.com/product-detail/C71629.html; LCSC PN (none) -> C71629
- C14, C15, C17: LCSC (none) -> https://www.lcsc.com/product-detail/C82453.html; LCSC PN (none) -> C82453
- C18, C19: LCSC (none) -> https://www.lcsc.com/product-detail/C76950.html; LCSC PN (none) -> C76950
- IC4: LCSC (none) -> https://www.lcsc.com/product-detail/C41378174.html; LCSC PN (none) -> C41378174
- J13: LCSC (none) -> https://www.lcsc.com/product-detail/C22438121.html; LCSC PN (none) -> C22438121
- J2: LCSC (none) -> https://www.lcsc.com/product-detail/C160403.html; LCSC PN (none) -> C160403
- J3, J4: LCSC (none) -> https://www.lcsc.com/product-detail/C189891.html; LCSC PN (none) -> C189891
- L1: LCSC (none) -> https://www.lcsc.com/product-detail/C42411119.html; LCSC PN (none) -> C42411119
- R10, R12: LCSC (none) -> https://www.lcsc.com/product-detail/C106235.html; LCSC PN (none) -> C106235
- R11: LCSC (none) -> https://www.lcsc.com/product-detail/C105871.html; LCSC PN (none) -> C105871
- R13: LCSC (none) -> https://www.lcsc.com/product-detail/C60490.html; LCSC PN (none) -> C60490
- R16, R17, R8: LCSC (none) -> https://www.lcsc.com/product-detail/C138002.html; LCSC PN (none) -> C138002
- R6, R7: LCSC (none) -> https://www.lcsc.com/product-detail/C226392.html; LCSC PN (none) -> C226392
- R9: LCSC (none) -> https://www.lcsc.com/product-detail/C105875.html; LCSC PN (none) -> C105875
- Y1: LCSC (none) -> https://www.lcsc.com/product-detail/C20625731.html; LCSC PN (none) -> C20625731
