File: hardware/csi.kicad_sch (KiCad schematic)
At the start: 1 part, among them J5 Conn_01x22_Female

Commit message: Small fixes
Parts:
- J5: Field4 Mouser -> (none); Field5 798-FH12-22S-0.5SH55 -> (none); Field6 FH12-22S-0.5SH55 -> (none); Field7 Hirose -> (none); MPN (none) -> FH12-22S-0.5SH(55); Manufacturer (none) -> Hirose; Mouser (none) -> https://www.mouser.com/ProductDetail/798-FH12-22S-0.5SH55; Mouser PN (none) -> 798-FH12-22S-0.5SH55; Part Description 22 Position FFC, FPC Connector Contacts, Bottom 0.020" (0.5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 -> (none)
Changed lines of the file:
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@@
 			)
 		)
-		(property "Datasheet" "https://www.hirose.com/product/document?clcode=&productname=&series=FH12&documenttype=Catalog&lang=en&documentid=D31648_en"
+		(property "Datasheet" "https://www.hirose.com/api/v1/products/CL0586-0532-7-55/documents/drawing_2d/content?lang=EN"
 			(at 41.91 45.72 0)
 			(hide yes)
@@
 			)
 		)
-		(property "Description" ""
+		(property "Description" "CONN FPC 22P 0.5mm bottom contact ZIF R/A"
 			(at 41.91 45.72 0)
 			(hide yes)
@@
 			)
 		)
-		(property "Field4" "Mouser"
+		(property "Manufacturer" "Hirose"
 			(at 41.91 45.72 0)
 			(hide yes)
@@
 			)
 		)
-		(property "Field5" "798-FH12-22S-0.5SH55"
+		(property "MPN" "FH12-22S-0.5SH(55)"
 			(at 41.91 45.72 0)
 			(hide yes)
@@
 			)
 		)
-		(property "Field6" "FH12-22S-0.5SH55"
+		(property "Mouser PN" "798-FH12-22S-0.5SH55"
 			(at 41.91 45.72 0)
 			(hide yes)
@@
 			)
 		)
-		(property "Field7" "Hirose"
+		(property "Mouser" "https://www.mouser.com/ProductDetail/798-FH12-22S-0.5SH55"
 			(at 41.91 45.72 0)
 			(hide yes)
-			(show_name no)
-			(do_not_autoplace no)
-			(effects
-				(font
-					(size 1.27 1.27)
-				)
-			)
-		)
-		(property "Part Description" "22 Position FFC, FPC Connector Contacts, Bottom 0.020\" (0.50mm) Surface Mount, Right Angle"
-			(at 41.91 45.72 0)
-			(hide yes)
