File: hardware/manafish.kicad_pcb (KiCad board)
At the start: 2 copper layers, 70 x 100 mm, 55 parts, among them IC1 BMI270, IC2 SHT45-AD1F-R2, J1 Conn_01x04_Pin, J2 SM03B-SRSS-TB, J3 AM32_1, J4 AM32_2, J5 Conn_01x22_Female, J6 Battery, J7 Conn_02x07_Odd_Even, J8 USB_C_Receptacle_USB2.0_14P, J9 THD-02-R, U1 TPD4EUSB30, U2 TPD4EUSB30, U3 MagJack-A70-112-331N126, U4 RP2354A, Y1 ABM8-272-T3

Commit message: Add rudimenatry poe module
Parts:
- removed J9: THD-02-R, Connector_PinHeader_2.54mm:PinHeader_2x02_P2.54mm_Vertical
- added R18: 4.7kR, Resistor_SMD:R_0402_1005Metric, B.Cu at (138.2, 69.4)
- added R19: 4.7kR, Resistor_SMD:R_0402_1005Metric, B.Cu at (140.2, 69.4)
- added U5: Ag5724-LPB, Silvertel:Silvertel_Ag5700-LPB, B.Cu at (123.3, 86.4)
Connections:
- IC1 pad 13: /I2C Peripherals/I2C1_SCL -> /I2C Peripherals/I2C0_SCL
- IC1 pad 14: /I2C Peripherals/I2C1_SDA -> /I2C Peripherals/I2C0_SDA
- U4 pad 5: unconnected-(U4-GPIO3-Pad5) -> /I2C Peripherals/I2C0_SCL
- U4 pad 7: unconnected-(U4-GPIO4-Pad7) -> /I2C Peripherals/I2C0_SDA
